File: hardware/banana-split.brd (EAGLE design)
At the start: 140.8 x 20.7 mm, 45 parts, among them IC1 REG1117, IC2 4050D, IC3 PIC12F1822SO08, IC4 6N138, X1 DIN5PIN, X2 DIN5PIN, X3 DIN5PIN, X4 DIN5PIN, X5 DIN5PIN, X6 DIN5PIN, X7 VERTICAL_3_5MM_SOCKET

Commit message: V5 PCB
Parts:
- removed IC5: (no value), microbuilder:SOIC-4
- added A, B, C, D, E: 1k8, rcl:R0603
- added C7: 100n, rcl:C0805
- added D2, D3, D4, D5: (no value), adafruit:SOD-123
- added R24: 1k8, rcl:R0805
Connections:
- new net N$26: C.1, D.1, X7.3
- new net N$29: E.1, X7.2
- new net N$30: A.1, B.1, C7.2, R24.2, X7.4
- net GND: now also C7.1, D3.A, D5.A, E.2; no longer IC5.-
- net MIDI_OUT: now also R24.1
- net N$20: now also B.2, C.2; no longer X7.4
- net N$24: now also A.2, D.2; no longer X7.3
- net N$27: now also D4.A, D5.C; no longer IC5.~1
- net N$28: now also D2.A, D3.C; no longer IC5.~2
- net VIN: now also D2.C, D4.C; no longer IC5.+
Routing:
- net MIDI_OUT: track 4.98 -> 39.2 mm
- net N$24: track 20.2 -> 49.1 mm, vias 0 -> 2
- net N$30: track 0.00 -> 21.0 mm
- net N$26: track 0.00 -> 14.2 mm, vias 0 -> 1
- net N$27: track 26.5 -> 38.9 mm, vias 0 -> 1
- net VIN: track 14.4 -> 26.6 mm
- net GND: track 24.1 -> 16.3 mm, vias 8 -> 10
- net N$28: track 28.4 -> 34.6 mm, vias 0 -> 1
- net N$29: track 0.00 -> 3.65 mm
- net N$20: track 22.0 -> 20.6 mm
- net MIDI_IN: track 81.3 -> 82.6 mm
- net N$7: track 41.3 -> 40.8 mm
Other:
- board text added: "rev 5"
- board text removed: "rev 4"

Commit message: v6 candidate
Parts:
- added CK, GD, GND: (no value), pinhead:1X01
- added F: JH_JP, jason_eagle6:JH_JP
- A, B, C, D, E: value 1k8 -> JH_JP; device rcl:R0603 -> jason_eagle6:JH_JP
- moved C7 13.4 mm to (29.8, 18.8), turned to 0 degrees
- moved RA2 3.56 mm to (42.8, 10.2), flipped to the top
- moved R24 1.58 mm to (22.7, 17.8), turned to 90 degrees
- moved B 0.71 mm to (3.68, 14.4), turned to 180 degrees
- moved A 0.65 mm to (3.68, 16.5), turned to 180 degrees
- moved C 0.53 mm to (3.68, 12.2), turned to 180 degrees
- moved E 0.38 mm to (7.62, 10.0)
- moved D 0.25 mm to (3.68, 10.0), turned to 180 degrees
- flipped RA4 to the top
Connections:
- new net N$31: C7.2, CK.1, F.P$1, R24.2
- net GND: now also E.P$1, GD.1, GND.1; no longer E.2
- net N$20: now also B.P$1, C.P$1; no longer B.2, C.2
- net N$24: now also A.P$1, D.P$1; no longer A.2, D.2
- net N$26: now also C.P$2, D.P$2, F.P$2; no longer C.1, D.1
- net N$29: now also E.P$2; no longer E.1
- net N$30: now also A.P$2, B.P$2; no longer A.1, B.1, C7.2, R24.2
Routing:
- net N$31: track 0.00 -> 11.8 mm
- net N$30: track 21.0 -> 9.50 mm
- net N$26: track 14.2 -> 20.1 mm
- net MIDI_OUT: track 39.2 -> 36.4 mm
- net N$25: track 1.94 -> 4.42 mm
- net N$24: track 49.1 -> 47.1 mm, vias 2 -> 1
- net N$20: track 20.6 -> 21.4 mm, vias 0 -> 2
- net N$29: track 3.65 -> 4.26 mm
Other:
- board text added: "rev 6"
- board text removed: "rev 5"

Commit message: V7 PCB
Parts:
- removed GD: (no value), pinhead:1X01
- A, B, C, D, E, F: value JH_JP -> 1k8; device jason_eagle6:JH_JP -> rcl:R0805
- moved E 12.3 mm to (16.2, 18.8), turned to 0 degrees
- moved F 8.39 mm to (10.2, 13.5), turned to 180 degrees
- moved A 1.85 mm to (5.08, 17.7)
- moved B 1.66 mm to (5.08, 15.2)
- moved C 1.49 mm to (5.08, 12.7)
- moved D 1.40 mm to (5.08, 10.2)
Connections:
- net GND: now also F.1; no longer E.P$1, GD.1
- net N$20: now also B.1, C.1; no longer B.P$1, C.P$1
- net N$24: now also A.1, D.1; no longer A.P$1, D.P$1
- net N$26: now also C.2, D.2; no longer C.P$2, D.P$2, F.P$2
- net N$29: now also F.2; no longer E.P$2
- net N$30: now also A.2, B.2, E.2; no longer A.P$2, B.P$2
- net N$31: now also E.1; no longer F.P$1
Routing:
- net N$26: track 20.1 -> 14.2 mm
- net N$24: track 47.1 -> 50.3 mm
- net N$30: track 9.50 -> 12.6 mm
- net N$20: track 21.4 -> 22.8 mm
Other:
- board text added: "rev 7"
- board text removed: "rev 6"
